Commit message: add icart_decription finish show multi i-cart

File: icart_description/urdf/icart_first.urdf (robot description, URDF)
Before this commit: robot icart, 6 links, 5 joints
Links:
- removed link base_footprint
- removed link base_link
- removed link caster_link
- removed link hokuyo_link
- removed link left_wheel_link
- removed link right_wheel_link
- added link base_footprint_first
- added link base_link_first, mass 0.500; collision mesh filename=package://icart_description/mesh/DAE/i-Cart_body.dae; visual mesh filename=package://icart_description/mesh/DAE/i-Cart_body.dae
- added link caster_link_first, mass 0.500; collision mesh filename=package://icart_description/mesh/DAE/i-Cart_caster.dae; visual mesh filename=package://icart_description/mesh/DAE/i-Cart_caster.dae
- added link hokuyo_link_first, mass 1e-5; collision box size=0.1 0.1 0.1; visual mesh filename=package://rrbot_description/meshes/hokuyo.dae
- added link left_wheel_link_first, mass 0.500; collision cylinder length=0.01 radius=0.0325; visual cylinder length=0.01 radius=0.0325
- added link right_wheel_link_first, mass 0.500; collision cylinder length=0.01 radius=0.0325; visual cylinder length=0.01 radius=0.0325
Joints:
- removed joint base_link_joint
- removed joint caster_joint
- removed joint hokuyo_joint
- removed joint left_wheel_joint
- removed joint right_wheel_joint
- added joint base_link_joint_first: type fixed, parent base_footprint_first, child base_link_first, origin xyz=-0.105 0 0.0545
- added joint caster_joint_first: type fixed, parent base_link_first, child caster_link_first, origin xyz=-0.096 0 -0.019 rpy=0 0 0
- added joint hokuyo_joint_first: type fixed, parent base_link_first, child hokuyo_link_first, origin xyz=0.105 0 0.035 rpy=0 0 0, axis 0 1 0
- added joint left_wheel_joint_first: type continuous, parent base_link_first, child left_wheel_link_first, origin xyz=0.105 0.178 -0.022 rpy=-1.5707 0 0, axis 0 0 1
- added joint right_wheel_joint_first: type continuous, parent base_link_first, child right_wheel_link_first, origin xyz=0.105 -0.178 -0.022 rpy=-1.5707 0 0, axis 0 0 1

File: icart_description/urdf/icart_second.urdf (robot description, URDF)
Before this commit: robot icart, 6 links, 5 joints
Links:
- removed link base_footprint
- removed link base_link
- removed link caster_link
- removed link hokuyo_link
- removed link left_wheel_link
- removed link right_wheel_link
- added link base_footprint_second
- added link base_link_second, mass 0.500; collision mesh filename=package://icart_description/mesh/DAE/i-Cart_body.dae; visual mesh filename=package://icart_description/mesh/DAE/i-Cart_body.dae
- added link caster_link_second, mass 0.500; collision mesh filename=package://icart_description/mesh/DAE/i-Cart_caster.dae; visual mesh filename=package://icart_description/mesh/DAE/i-Cart_caster.dae
- added link hokuyo_link_second, mass 1e-5; collision box size=0.1 0.1 0.1; visual mesh filename=package://rrbot_description/meshes/hokuyo.dae
- added link left_wheel_link_second, mass 0.500; collision cylinder length=0.01 radius=0.0325; visual cylinder length=0.01 radius=0.0325
- added link right_wheel_link_second, mass 0.500; collision cylinder length=0.01 radius=0.0325; visual cylinder length=0.01 radius=0.0325
Joints:
- removed joint base_link_joint
- removed joint caster_joint
- removed joint hokuyo_joint
- removed joint left_wheel_joint
- removed joint right_wheel_joint
- added joint base_link_joint_second: type fixed, parent base_footprint_second, child base_link_second, origin xyz=-0.105 0 0.545
- added joint caster_joint_second: type fixed, parent base_link_second, child caster_link_second, origin xyz=-0.096 0 -0.019 rpy=0 0 0
- added joint hokuyo_joint_second: type fixed, parent base_link_second, child hokuyo_link_second, origin xyz=0.105 0 0.035 rpy=0 0 0, axis 0 1 0
- added joint left_wheel_joint_second: type continuous, parent base_link_second, child left_wheel_link_second, origin xyz=0.105 0.178 -0.022 rpy=-1.5707 0 0, axis 0 0 1
- added joint right_wheel_joint_second: type continuous, parent base_link_second, child right_wheel_link_second, origin xyz=0.105 -0.178 -0.022 rpy=-1.5707 0 0, axis 0 0 1

Commit message: gmappingとamclの同時起動に成功した

File: icart_description/urdf/icart_first.urdf (robot description, URDF)
Before this commit: robot icart_first, 6 links, 5 joints
Links:
- removed link base_footprint_first
Joints:
- removed joint base_link_joint_first

File: icart_description/urdf/icart_second.urdf (robot description, URDF)
Before this commit: robot icart_second, 6 links, 5 joints
Links:
- removed link base_footprint_second
Joints:
- removed joint base_link_joint_second

Commit message: マップ上から位置取得

File: icart_description/urdf/icart_first.urdf (robot description, URDF)
Before this commit: robot icart_first, 5 links, 4 joints
Links:
- added link base_footprint_first
Joints:
- added joint base_link_joint_first: type fixed, parent base_link_first, child base_footprint_first, origin xyz=0.105 0 0.0

File: icart_description/urdf/icart_second.urdf (robot description, URDF)
Before this commit: robot icart_second, 5 links, 4 joints
Links:
- added link base_footprint_second
Joints:
- added joint base_link_joint_second: type fixed, parent base_link_second, child base_footprint_second, origin xyz=0.105 0 0.0

Commit message: URGの向きを逆向き レーザを見えなくする

File: icart_description/urdf/icart_first.urdf (robot description, URDF)
Before this commit: robot icart_first, 5 links, 4 joints
Joints:
- joint hokuyo_joint_first: axis 0 1 0 -> 0 0 0; origin xyz=0.105 0 0.035 rpy=0 0 0 -> xyz=0.105 0 0.135 rpy=0 0 3.14

File: icart_description/urdf/icart_second.urdf (robot description, URDF)
Before this commit: robot icart_second, 5 links, 4 joints
Joints:
- joint hokuyo_joint_second: axis 0 1 0 -> 0 0 0; origin xyz=0.105 0 0.035 rpy=0 0 0 -> xyz=0.105 0 0.135 rpy=0 0 3.14

Commit message: URGの向きを元に戻した

File: icart_description/urdf/icart_first.urdf (robot description, URDF)
Before this commit: robot icart_first, 5 links, 4 joints
Joints:
- joint hokuyo_joint_first: origin xyz=0.105 0 0.135 rpy=0 0 3.14 -> xyz=0.105 0 0.135 rpy=0 0 0

File: icart_description/urdf/icart_second.urdf (robot description, URDF)
Before this commit: robot icart_second, 5 links, 4 joints
Joints:
- joint hokuyo_joint_second: origin xyz=0.105 0 0.135 rpy=0 0 3.14 -> xyz=0.105 0 0.135 rpy=0 0 0

Commit message: モデルを簡単にしたのと，真値を取得できるようにした

File: icart_description/urdf/icart_first.urdf (robot description, URDF)
Before this commit: robot icart_first, 5 links, 4 joints
Links:
- added link base_foot_print_first
- added link base_link_first_offset
- link base_link_first: mass 0.000 -> ${base_mass}; geometry collision box size=${bd} ${bw} ${bh}; visual box size=${bd} ${bw} ${bh}
- link caster_link_first: mass 5.500 -> ${caster_mass}; geometry collision sphere radius=${cr}; visual sphere radius=${cr}
- link left_wheel_link_first: mass 10.500 -> ${wheel_mass}; geometry collision cylinder length=${wl} radius=${wr}; visual cylinder length=${wl} radius=${wr}
- link right_wheel_link_first: mass 10.500 -> ${wheel_mass}; geometry collision cylinder length=${wl} radius=${wr}; visual cylinder length=${wl} radius=${wr}
Joints:
- added joint foot_print_first: type fixed, parent base_foot_print_first, child base_link_first, origin xyz=-0.105 0 ${cr} rpy=0 0 0
- added joint offset_first: type fixed, parent base_link_first, child base_link_first_offset, origin xyz=-0.055 0 0 rpy=0 0 0
- joint caster_joint_first: origin xyz=-0.096 0 -0.019 rpy=0 0 0 -> xyz=-0.096 0 0 rpy=0 0 0
- joint hokuyo_joint_first: origin xyz=0.105 0 0.135 rpy=0 0 0 -> xyz=0 0 0.135 rpy=0 0 0; parent base_link_first -> base_foot_print_first
- joint left_wheel_joint_first: origin xyz=0.105 0.178 -0.022 rpy=-1.5707 0 0 -> xyz=0.105 0.178 0 rpy=-1.5707 0 0
- joint right_wheel_joint_first: origin xyz=0.105 -0.178 -0.022 rpy=1.5707 0 0 -> xyz=0.105 -0.178 0 rpy=1.5707 0 0

File: icart_description/urdf/icart_second.urdf (robot description, URDF)
Before this commit: robot icart_second, 5 links, 4 joints
Links:
- added link base_foot_print_second
- added link base_link_second_offset
- link base_link_second: mass 0.000 -> ${base_mass}; geometry collision box size=${bd} ${bw} ${bh}; visual box size=${bd} ${bw} ${bh}
- link caster_link_second: mass 5.500 -> ${caster_mass}; geometry collision sphere radius=${cr}; visual sphere radius=${cr}
- link left_wheel_link_second: mass 10.500 -> ${wheel_mass}; geometry collision cylinder length=${wl} radius=${wr}; visual cylinder length=${wl} radius=${wr}
- link right_wheel_link_second: mass 10.500 -> ${wheel_mass}; geometry collision cylinder length=${wl} radius=${wr}; visual cylinder length=${wl} radius=${wr}
Joints:
- added joint foot_print_second: type fixed, parent base_foot_print_second, child base_link_second, origin xyz=-0.105 0 ${cr} rpy=0 0 0
- added joint offset_second: type fixed, parent base_link_second, child base_link_second_offset, origin xyz=-0.055 0 0 rpy=0 0 0
- joint caster_joint_second: origin xyz=-0.096 0 -0.019 rpy=0 0 0 -> xyz=-0.096 0 0 rpy=0 0 0
- joint hokuyo_joint_second: origin xyz=0.105 0 0.135 rpy=0 0 0 -> xyz=0 0 0.135 rpy=0 0 0; parent base_link_second -> base_foot_print_second
- joint left_wheel_joint_second: origin xyz=0.105 0.178 -0.022 rpy=-1.5707 0 0 -> xyz=0.105 0.178 0 rpy=-1.5707 0 0
- joint right_wheel_joint_second: origin xyz=0.105 -0.178 -0.022 rpy=1.5707 0 0 -> xyz=0.105 -0.178 0 rpy=1.5707 0 0

Commit message: URGの位置と性能変更

File: icart_description/urdf/icart_first.urdf (robot description, URDF)
Before this commit: robot icart_first, 7 links, 6 joints
Joints:
- joint hokuyo_joint_first: origin xyz=0 0 0.135 rpy=0 0 0 -> xyz=0 0 0.0825 rpy=0 0 3.141592

File: icart_description/urdf/icart_second.urdf (robot description, URDF)
Before this commit: robot icart_second, 7 links, 6 joints
Joints:
- joint hokuyo_joint_second: origin xyz=0 0 0.135 rpy=0 0 0 -> xyz=0 0 0.0825 rpy=0 0 3.141592

Commit message: icartに搬送物の支持点を追加

File: icart_description/urdf/icart_first.urdf (robot description, URDF)
Before this commit: robot icart_first, 7 links, 6 joints
Links:
- added link stick_first, mass ${stick_mass}; collision box size=${sd} ${sw} ${sh}; visual box size=${sd} ${sw} ${sh}
- added link stopper1_first, mass ${stopper_mass}; collision box size=${stopper_d} ${stopper_w} ${stopper_h}; visual box size=${stopper_d} ${stopper_w} ${stopper_h}
- added link stopper2_first, mass ${stopper_mass}; collision box size=${stopper_d} ${stopper_w} ${stopper_h}; visual box size=${stopper_d} ${stopper_w} ${stopper_h}
- added link stopper3_first, mass ${stopper_mass}; collision box size=${stopper_d} ${stopper_w} ${stopper_h}; visual box size=${stopper_d} ${stopper_w} ${stopper_h}
- added link table_first, mass ${table_mass}; collision cylinder length=${tl} radius=${tr}; visual cylinder length=${tl} radius=${tr}
Joints:
- added joint stick_joint_first: type fixed, parent base_link_first_offset, child stick_first, origin xyz=0 0 ${sh/2+bh/2} rpy=0 0 0
- added joint stopper1_joint_first: type fixed, parent table_first, child stopper1_first, origin xyz=0 ${-tr/2} ${tl/2+stopper_h/2} rpy=0 0 0
- added joint stopper2_joint_first: type fixed, parent table_first, child stopper2_first, origin xyz=0 ${tr/2} ${tl/2+stopper_h/2} rpy=0 0 0
- added joint stopper3_joint_first: type fixed, parent table_first, child stopper3_first, origin xyz=${tr/2} 0 ${tl/2+stopper_h/2} rpy=0 0 1.57
- added joint table_joint_first: type continuous, parent stick_first, child table_first, origin xyz=0 0 ${tl/2+sh/2} rpy=0 0 0, axis 0 0 1

File: icart_description/urdf/icart_second.urdf (robot description, URDF)
Before this commit: robot icart_second, 7 links, 6 joints
Links:
- added link stick_second, mass ${stick_mass}; collision box size=${sd} ${sw} ${sh}; visual box size=${sd} ${sw} ${sh}
- added link stopper1_second, mass ${stopper_mass}; collision box size=${stopper_d} ${stopper_w} ${stopper_h}; visual box size=${stopper_d} ${stopper_w} ${stopper_h}
- added link stopper2_second, mass ${stopper_mass}; collision box size=${stopper_d} ${stopper_w} ${stopper_h}; visual box size=${stopper_d} ${stopper_w} ${stopper_h}
- added link stopper3_second, mass ${stopper_mass}; collision box size=${stopper_d} ${stopper_w} ${stopper_h}; visual box size=${stopper_d} ${stopper_w} ${stopper_h}
- added link table_second, mass ${table_mass}; collision cylinder length=${tl} radius=${tr}; visual cylinder length=${tl} radius=${tr}
Joints:
- added joint stick_second: type fixed, parent base_link_second_offset, child stick_second, origin xyz=0 0 ${sh/2+bh/2} rpy=0 0 0
- added joint stopper1_joint_second: type fixed, parent table_second, child stopper1_second, origin xyz=0 ${-tr/2} ${tl/2+stopper_h/2} rpy=0 0 0
- added joint stopper2_joint_second: type fixed, parent table_second, child stopper2_second, origin xyz=0 ${tr/2} ${tl/2+stopper_h/2} rpy=0 0 0
- added joint stopper3_joint_second: type fixed, parent table_second, child stopper3_second, origin xyz=${-tr/2} 0 ${tl/2+stopper_h/2} rpy=0 0 1.57
- added joint table_joint_second: type continuous, parent stick_second, child table_second, origin xyz=0 0 ${tl/2+sh/2} rpy=0 0 0, axis 0 0 1

Commit message: wheelの重さを変更

File: icart_description/urdf/icart_first.urdf (robot description, URDF)
Before this commit: robot icart_first, 12 links, 11 joints
Links:
- removed link stopper1_first
- removed link stopper2_first
- removed link stopper3_first
Joints:
- removed joint stopper1_joint_first
- removed joint stopper2_joint_first
- removed joint stopper3_joint_first

File: icart_description/urdf/icart_second.urdf (robot description, URDF)
Before this commit: robot icart_second, 12 links, 11 joints
Links:
- removed link stopper1_second
- removed link stopper2_second
- removed link stopper3_second
Joints:
- removed joint stopper1_joint_second
- removed joint stopper2_joint_second
- removed joint stopper3_joint_second

Commit message: 連結部分を追加したモデルを作成

File: icart_description/urdf/icart_first.urdf (robot description, URDF)
Before this commit: robot icart_first, 9 links, 8 joints
Links:
- link stick_first: geometry collision cylinder length=${sl} radius=${sr}; visual cylinder length=${sl} radius=${sr}
Joints:
- joint table_joint_first: origin xyz=0 0 ${tl/2+sh/2} rpy=0 0 0 -> xyz=0 0 ${tl/2} rpy=0 0 0

File: icart_description/urdf/icart_second.urdf (robot description, URDF)
Before this commit: robot icart_second, 9 links, 8 joints
Links:
- link stick_second: geometry collision cylinder length=${sl} radius=${sr}; visual cylinder length=${sl} radius=${sr}
Joints:
- joint table_joint_second: origin xyz=0 0 ${tl/2+sh/2} rpy=0 0 0 -> xyz=0 0 ${tl/2} rpy=0 0 0
