Commit message: link部分に見やすいようにマークを追加

File: icart_description/urdf/linking.urdf (robot description, URDF)
Before this commit: robot linking, 9 links, 8 joints
Links:
- added link mark, mass ${mmass}; collision cylinder length=${mh} radius=${mr}; visual cylinder length=${mh} radius=${mr}
Joints:
- added joint marker_joint: type fixed, parent block, child mark, origin xyz=0 0 ${(mh/2)+(h/2)} rpy=0 0 0
