Commit message: add single_simulation

File: icart_description/urdf/icart.urdf (robot description, URDF)
Before this commit: robot icart, 6 links, 5 joints
Joints:
- joint base_link_joint: origin xyz=-0.10 0 0.050 -> xyz=-0.105 0 0.0545

File: icart_description/urdf/icart_second.urdf (robot description, URDF)
Before this commit: robot icart_second, 6 links, 5 joints
Joints:
- joint base_link_joint_second: origin xyz=-0.105 0 0.545 -> xyz=-0.105 0 0.0545

Commit message: finish gazebo_multi_control.launch

File: icart_description/urdf/icart.urdf (robot description, URDF)
Before this commit: robot icart, 6 links, 5 joints
Joints:
- joint right_wheel_joint: axis 0 0 1 -> 0 0 -1; origin xyz=0.105 -0.178 -0.022 rpy=-1.5707 0 0 -> xyz=0.105 -0.178 -0.022 rpy=1.5707 0 0

File: icart_description/urdf/icart_second.urdf (robot description, URDF)
Before this commit: robot icart_second, 6 links, 5 joints
Links:
- link base_link_second: mass 0.500 -> 0.000
- link caster_link_second: geometry collision mesh filename=package://icart_description/mesh/DAE/i-Cart_caster.dae; visual sphere radius=0.0325
- link left_wheel_link_second: mass 0.500 -> 1.500
- link right_wheel_link_second: mass 0.500 -> 1.500
Joints:
- joint right_wheel_joint_second: axis 0 0 1 -> 0 0 -1; origin xyz=0.105 -0.178 -0.022 rpy=-1.5707 0 0 -> xyz=0.105 -0.178 -0.022 rpy=1.5707 0 0

File: icart_description/urdf/simple_icart.urdf (robot description, URDF)
Before this commit: robot icart_first, 6 links, 5 joints
Links:
- removed link base_footprint_first
- removed link base_link_first
- removed link caster_link_first
- removed link hokuyo_link_first
- removed link left_wheel_link_first
- removed link right_wheel_link_first
- added link base_footprint
- added link base_link, mass 0.500; collision box size=0.280 0.340 0.030; visual box size=0.280 0.340 0.030
- added link caster_link, mass 0.500; collision sphere radius=0.0325; visual sphere radius=0.0325
- added link hokuyo_link, mass 1e-5; collision box size=0.1 0.1 0.1; visual mesh filename=package://rrbot_description/meshes/hokuyo.dae
- added link left_wheel_link, mass 0.500; collision cylinder length=0.01 radius=0.0325; visual cylinder length=0.01 radius=0.0325
- added link right_wheel_link, mass 0.500; collision cylinder length=0.01 radius=0.0325; visual cylinder length=0.01 radius=0.0325
Joints:
- removed joint base_link_joint_first
- removed joint caster_joint_first
- removed joint hokuyo_joint_first
- removed joint left_wheel_joint_first
- removed joint right_wheel_joint_first
- added joint base_link_joint: type fixed, parent base_footprint, child base_link, origin xyz=-0.105 0 -0.0325
- added joint caster_joint: type fixed, parent base_link, child caster_link, origin xyz=-0.096 0 0.0 rpy=0 0 0
- added joint hokuyo_joint: type fixed, parent base_link, child hokuyo_link, origin xyz=0.105 0 0.055 rpy=0 0 0, axis 0 1 0
- added joint left_wheel_joint: type continuous, parent base_link, child left_wheel_link, origin xyz=0.105 0.178 0 rpy=-1.5707 0 0, axis 0 0 1
- added joint right_wheel_joint: type continuous, parent base_link, child right_wheel_link, origin xyz=0.105 -0.178 0 rpy=1.5707 0 0, axis 0 0 -1

Commit message: 修士前のデータ保管

File: icart_description/urdf/icart.urdf (robot description, URDF)
Before this commit: robot icart, 6 links, 5 joints
Links:
- link hokuyo_link: geometry visual mesh filename=package://rrbot_description/meshes/hokuyo.dae

File: icart_description/urdf/icart_first.urdf (robot description, URDF)
Before this commit: robot icart_first, 6 links, 5 joints
Links:
- link caster_link_first: mass 0.500 -> 5.500
- link hokuyo_link_first: geometry visual mesh filename=package://rrbot_description/meshes/hokuyo.dae
- link left_wheel_link_first: mass 1.500 -> 10.500
- link right_wheel_link_first: mass 1.500 -> 10.500

File: icart_description/urdf/icart_second.urdf (robot description, URDF)
Before this commit: robot icart_second, 6 links, 5 joints
Links:
- link caster_link_second: mass 0.500 -> 5.500
- link hokuyo_link_second: geometry visual mesh filename=package://rrbot_description/meshes/hokuyo.dae
- link left_wheel_link_second: mass 1.500 -> 10.500
- link right_wheel_link_second: mass 1.500 -> 10.500

Commit message: linkのタイポを修正

File: icart_description/urdf/icart.urdf (robot description, URDF)
Before this commit: robot icart, 6 links, 5 joints
Links:
- removed link base_footprint
- added link base_foot_print
Joints:
- joint base_link_joint: parent base_footprint -> base_foot_print

Commit message: モデルを修正

File: icart_description/urdf/icart.urdf (robot description, URDF)
Before this commit: robot icart, 6 links, 5 joints
Links:
- added link base_link_offset
- added link stick, mass ${stick_mass}; collision cylinder length=${sl} radius=${sr}; visual cylinder length=${sl} radius=${sr}
- added link table, mass ${table_mass}; collision cylinder length=${tl} radius=${tr}; visual cylinder length=${tl} radius=${tr}
- link base_link: mass 0.500 -> ${base_mass}; geometry collision box size=${bd} ${bw} ${bh}; visual box size=${bd} ${bw} ${bh}
- link caster_link: mass 0.500 -> ${caster_mass}; geometry collision sphere radius=${cr}; visual sphere radius=${cr}
- link left_wheel_link: mass 0.500 -> ${wheel_mass}; geometry collision cylinder length=${wl} radius=${wr}; visual cylinder length=${wl} radius=${wr}
- link right_wheel_link: mass 0.500 -> ${wheel_mass}; geometry collision cylinder length=${wl} radius=${wr}; visual cylinder length=${wl} radius=${wr}
Joints:
- removed joint base_link_joint
- added joint foot_print: type fixed, parent base_foot_print, child base_link, origin xyz=-0.105 0 ${cr} rpy=0 0 0
- added joint offset: type fixed, parent base_link, child base_link_offset, origin xyz=-0.055 0 0 rpy=0 0 0
- added joint stick_joint: type fixed, parent base_link_offset, child stick, origin xyz=0 0 ${sh/2+bh/2} rpy=0 0 0
- added joint table_joint: type continuous, parent stick, child table, origin xyz=0 0 ${tl/2} rpy=0 0 0, axis 0 0 1
- joint caster_joint: origin xyz=-0.096 0 -0.019 rpy=0 0 0 -> xyz=-0.096 0 0 rpy=0 0 0
- joint hokuyo_joint: axis 0 1 0 -> 0 0 0; origin xyz=0.105 0 0.035 rpy=0 0 0 -> xyz=0 0 0.0825 rpy=0 0 3.141592; parent base_link -> base_foot_print
- joint left_wheel_joint: origin xyz=0.105 0.178 -0.022 rpy=-1.5707 0 0 -> xyz=0.105 0.178 0 rpy=-1.5707 0 0
- joint right_wheel_joint: origin xyz=0.105 -0.178 -0.022 rpy=1.5707 0 0 -> xyz=0.105 -0.178 0 rpy=1.5707 0 0

Commit message: LRFの向きを修正

File: icart_description/urdf/icart.urdf (robot description, URDF)
Before this commit: robot icart, 9 links, 8 joints
Joints:
- joint hokuyo_joint: origin xyz=0 0 0.0825 rpy=0 0 3.141592 -> xyz=0 0 0.0825 rpy=0 0 0
