Commit message: rvizにdepthカメラのポイントクラウド表示できた そもそもgazeboにバグがあってカメラのtfを回転させてもポイントクラウドが違う方に回転する だから，余分にjointを作って回転させる

File: icart_description/urdf/icart_depth.urdf (robot description, URDF)
Before this commit: robot icart_depth, 10 links, 9 joints
Links:
- removed link camera_link
- added link pico_flexx_depth_frame
- added link pico_flexx_link, mass 0.001; collision box size=0.007 0.066 0.016; visual box size=0.007 0.066 0.016
- added link pico_flexx_link_optical_frame
Joints:
- removed joint depth_joint
- added joint pico_flexx_base_joint: type fixed, parent base_foot_print, child pico_flexx_link_optical_frame, origin xyz=0.2 0 0.07 rpy=0 0 0
- added joint pico_flexx_depth_joint: type fixed, parent pico_flexx_link_optical_frame, child pico_flexx_depth_frame, origin xyz=0 0 0 rpy=${-M_PI/2} 0 ${-M_PI/2}
- added joint pico_flexx_joint: type fixed, parent pico_flexx_link_optical_frame, child pico_flexx_link, origin xyz=0 0 0 rpy=0 0 0

Commit message: depthのカメラの実装が出来た

File: icart_description/urdf/icart_depth.urdf (robot description, URDF)
Before this commit: robot icart_depth, 12 links, 11 joints
Links:
- removed link pico_flexx_depth_frame
- removed link pico_flexx_link
- removed link pico_flexx_link_optical_frame
- added link depth_camera_base_link
- added link depth_camera_link, mass 0.001; collision box size=0.007 0.066 0.016; visual box size=0.007 0.066 0.016
- added link depth_camera_rviz_link
Joints:
- removed joint pico_flexx_base_joint
- removed joint pico_flexx_depth_joint
- removed joint pico_flexx_joint
- added joint depth_camera_base_joint: type fixed, parent base_foot_print, child depth_camera_base_link, origin xyz=0 0 0.2 rpy=0 0 0
- added joint depth_camera_joint: type fixed, parent depth_camera_base_link, child depth_camera_link, origin xyz=0 0 0 rpy=0 0 0
- added joint depth_camera_rviz_joint: type fixed, parent depth_camera_base_link, child depth_camera_rviz_link, origin xyz=0 0 0 rpy=${-M_PI/2} 0 ${-M_PI/2}

Commit message: depthcameraにpan_tilt台を搭載

File: icart_description/urdf/icart_depth.urdf (robot description, URDF)
Before this commit: robot icart_depth, 12 links, 11 joints
Links:
- added link depth_pan_link
- added link depth_pan_tilt_link, mass 0.001
- added link depth_tilt_link
Joints:
- added joint depth_camera_pan_joint: type revolute, parent base_foot_print, child depth_pan_link, origin xyz=0 0 0.2 rpy=0 0 0, axis 0 0 1, limit lower=-3.14 upper=3.14 effort=30 velocity=1.571
- added joint depth_camera_pan_tilt_joint: type fixed, parent depth_pan_link, child depth_pan_tilt_link, origin xyz=0 0 0 rpy=0 0 0
- added joint depth_camera_tilt_joint: type revolute, parent depth_pan_tilt_link, child depth_tilt_link, origin xyz=0 0 0 rpy=0 0 0, axis 0 1 0, limit lower=-3.14 upper=3.14 effort=30 velocity=1.571
- joint depth_camera_base_joint: origin xyz=0 0 0.2 rpy=0 0 0 -> xyz=0 0 0.0 rpy=0 0 0; parent base_foot_print -> depth_tilt_link
